File: RaspberryPi.kicad_sch (KiCad schematic)
At the start: 72 parts, among them P1 USB_C_Plug_USB2.0, Q1 Si9430, U1 TPS7A0310, U2 TLV62565-LibCool, U3 TPS72118, U4 TPS62052DGS, U5 MAX1651, U6 TPS7A21

Commit message: 内存完工
Connections:
- net A0: now also U?.N3 (A0), U?.N3 (A0), U?.N3 (A0)
- net A1: now also U?.P7 (A1), U?.P7 (A1), U?.P7 (A1)
- net A10: now also U?.L7 (A10/AP), U?.L7 (A10/AP), U?.L7 (A10/AP)
- net A11: now also U?.R7 (A11), U?.R7 (A11), U?.R7 (A11)
- net A12: now also U?.N7 (A12/~{BC}), U?.N7 (A12/~{BC}), U?.N7 (A12/~{BC})
- net A13: now also U?.T3 (A13), U?.T3 (A13), U?.T3 (A13)
- net A14: now also U?.T7 (A14), U?.T7 (A14), U?.T7 (A14)
- net A2: now also U?.P3 (A2), U?.P3 (A2), U?.P3 (A2)
- net A3: now also U?.N2 (A3), U?.N2 (A3), U?.N2 (A3)
- net A4: now also U?.P8 (A4), U?.P8 (A4), U?.P8 (A4)
- net A5: now also U?.P2 (A5), U?.P2 (A5), U?.P2 (A5)
- net A6: now also U?.R8 (A6), U?.R8 (A6), U?.R8 (A6)
- net A7: now also U?.R2 (A7), U?.R2 (A7), U?.R2 (A7)
- net A8: now also U?.T8 (A8), U?.T8 (A8), U?.T8 (A8)
- net A9: now also U?.R3 (A9), U?.R3 (A9), U?.R3 (A9)
- net BA0: now also U?.M2 (BA0), U?.M2 (BA0), U?.M2 (BA0)
- net BA1: now also U?.N8 (BA1), U?.N8 (BA1), U?.N8 (BA1)
- net BA2: now also U?.M3 (BA2), U?.M3 (BA2), U?.M3 (BA2)
- net CASN: now also U?.K3 (~{CAS}), U?.K3 (~{CAS}), U?.K3 (~{CAS})
- net CKE0: now also U?.K9 (CKE), U?.K9 (CKE), U?.K9 (CKE)
- net CLK: now also U?.J7 (CK), U?.J7 (CK), U?.J7 (CK)
- net CLKN: now also U?.K7 (~{CK}), U?.K7 (~{CK}), U?.K7 (~{CK})
- net CS0N: now also U?.L2 (~{CS})
- net CS1N: now also U?.L2 (~{CS}), U?.L2 (~{CS})
- net D0: now also U?.F7 (DQ1)
- net D10: now also U?.F2 (DQ2), U?.F8 (DQ3)
- net D11: now also U?.F2 (DQ2), U?.F8 (DQ3)
- net D12: now also U?.H3 (DQ4), U?.H7 (DQ7)
- net D13: now also U?.G2 (DQ6), U?.H8 (DQ5)
- net D14: now also U?.G2 (DQ6), U?.H8 (DQ5)
- net D15: now also U?.H3 (DQ4), U?.H7 (DQ7)
- net D16: now also U?.C3 (DQ9)
- net D17: now also U?.D7 (DQ8)
- net D18: now also U?.C2 (DQ11)
- net D19: now also U?.C8 (DQ10)
- net D2: now also U?.F8 (DQ3)
- net D20: now also U?.A3 (DQ15)
- net D21: now also U?.B8 (DQ14)
- net D22: now also U?.A2 (DQ13)
- net D23: now also U?.A7 (DQ12)
- net D24: now also U?.C3 (DQ9), U?.D7 (DQ8)
- net D25: now also U?.C3 (DQ9), U?.D7 (DQ8)
- net D26: now also U?.C2 (DQ11), U?.C8 (DQ10)
- net D27: now also U?.C2 (DQ11), U?.C8 (DQ10)
- net D28: now also U?.A3 (DQ15), U?.A7 (DQ12)
- net D29: now also U?.A2 (DQ13), U?.B8 (DQ14)
- net D3: now also U?.F2 (DQ2)
- net D30: now also U?.A2 (DQ13), U?.B8 (DQ14)
- net D31: now also U?.A3 (DQ15), U?.A7 (DQ12)
- net D4: now also U?.H7 (DQ7)
- net D6: now also U?.H8 (DQ5)
- net D7: now also U?.H3 (DQ4)
- net D8: now also U?.E3 (DQ0), U?.F7 (DQ1)
- net D9: now also U?.E3 (DQ0), U?.F7 (DQ1)
- net DDRPWR: now also U?.A1 (VDDQ), U?.A1 (VDDQ), U?.A1 (VDDQ), U?.A8 (VDDQ), U?.A8 (VDDQ), U?.A8 (VDDQ), U?.B2 (VDD), U?.B2 (VDD), U?.B2 (VDD), U?.C1 (VDDQ), U?.C1 (VDDQ), U?.C1 (VDDQ), U?.C9 (VDDQ), U?.C9 (VDDQ), U?.C9 (VDDQ), U?.D2 (VDDQ), U?.D2 (VDDQ), U?.D2 (VDDQ), U?.D9 (VDD), U?.D9 (VDD), U?.D9 (VDD), U?.E9 (VDDQ), U?.E9 (VDDQ), U?.E9 (VDDQ), U?.F1 (VDDQ), U?.F1 (VDDQ), U?.F1 (VDDQ), U?.G7 (VDD), U?.G7 (VDD), U?.G7 (VDD), U?.H1 (VREFDQ), U?.H1 (VREFDQ), U?.H1 (VREFDQ), U?.H2 (VDDQ), U?.H2 (VDDQ), U?.H2 (VDDQ), U?.H9 (VDDQ), U?.H9 (VDDQ), U?.H9 (VDDQ), U?.K2 (VDD), U?.K2 (VDD), U?.K2 (VDD), U?.K8 (VDD), U?.K8 (VDD), U?.K8 (VDD), U?.M8 (VREFCA), U?.M8 (VREFCA), U?.M8 (VREFCA), U?.N1 (VDD), U?.N1 (VDD), U?.N1 (VDD), U?.N9 (VDD), U?.N9 (VDD), U?.N9 (VDD), U?.R1 (VDD), U?.R1 (VDD), U?.R1 (VDD), U?.R9 (VDD), U?.R9 (VDD), U?.R9 (VDD)
- net DDR_RST: now also U?.T2 (~{RESET}), U?.T2 (~{RESET}), U?.T2 (~{RESET})
- net DM0: now also U?.E7 (LDM)
- net DM1: now also U?.E7 (LDM), U?.E7 (LDM)
- net DM2: now also U?.D3 (UDM)
- net DM3: now also U?.D3 (UDM), U?.D3 (UDM)
- net DQS0M: now also U?.G3 (~{LDQS}), U?.G3 (~{LDQS}), U?.G3 (~{LDQS})
- net DQS0P: now also U?.F3 (LDQS)
- net DQS1P: now also U?.F3 (LDQS), U?.F3 (LDQS)
- net DQS2M: now also U?.B7 (~{UDQS})
- net DQS2P: now also U?.C7 (UDQS)
- net DQS3M: now also U?.B7 (~{UDQS}), U?.B7 (~{UDQS})
- net DQS3P: now also U?.C7 (UDQS), U?.C7 (UDQS)
- net GND: now also U?.A9 (VSS), U?.A9 (VSS), U?.A9 (VSS), U?.B1 (VSSQ), U?.B1 (VSSQ), U?.B1 (VSSQ), U?.B3 (VSS), U?.B3 (VSS), U?.B3 (VSS), U?.B9 (VSSQ), U?.B9 (VSSQ), U?.B9 (VSSQ), U?.D1 (VSSQ), U?.D1 (VSSQ), U?.D1 (VSSQ), U?.D8 (VSSQ), U?.D8 (VSSQ), U?.D8 (VSSQ), U?.E1 (VSS), U?.E1 (VSS), U?.E1 (VSS), U?.E2 (VSSQ), U?.E2 (VSSQ), U?.E2 (VSSQ), U?.E8 (VSSQ), U?.E8 (VSSQ), U?.E8 (VSSQ), U?.F9 (VSSQ), U?.F9 (VSSQ), U?.F9 (VSSQ), U?.G1 (VSSQ), U?.G1 (VSSQ), U?.G1 (VSSQ), U?.G8 (VSS), U?.G8 (VSS), U?.G8 (VSS), U?.G9 (VSSQ), U?.G9 (VSSQ), U?.G9 (VSSQ), U?.J2 (VSS), U?.J2 (VSS), U?.J2 (VSS), U?.J8 (VSS), U?.J8 (VSS), U?.J8 (VSS), U?.M1 (VSS), U?.M1 (VSS), U?.M1 (VSS), U?.M9 (VSS), U?.M9 (VSS), U?.M9 (VSS), U?.P1 (VSS), U?.P1 (VSS), U?.P1 (VSS), U?.P9 (VSS), U?.P9 (VSS), U?.P9 (VSS), U?.T1 (VSS), U?.T1 (VSS), U?.T1 (VSS), U?.T9 (VSS), U?.T9 (VSS), U?.T9 (VSS)
- net ODT0: now also U?.K1 (ODT)
- net ODT1: now also U?.K1 (ODT), U?.K1 (ODT)
- net RASN: now also U?.J3 (~{RAS}), U?.J3 (~{RAS}), U?.J3 (~{RAS})
- net WEN: now also U?.L3 (~{WE}), U?.L3 (~{WE}), U?.L3 (~{WE})
- no-connect marks 10 -> 13
Other:
- moved on the sheet: U?
