File: RaspberryPi.kicad_sch (KiCad schematic)
At the start: 267 parts, among them J1 DBG1, J2 USB_A, J3 Micro_SD_Card_Det, J4 RJ45, J5 USB_A, J6 USB_A, J7 USB_A, J8 HDMI_A, J9 DB9_Male, P1 USB_C_Plug_USB2.0, Q1 Si9430, Q2 2N7002, Q3 2N7002, Q4 2N7002, U1 TPS7A0310, U10 RK3368_DDR, U11 RK3368_SYS, U12 MT41KxxxM16TW, U13 MT41KxxxM16TW, U14 MT41KxxxM16TW, U15 MT41KxxxM16TW, U16 RK3368_UART, U17 RK3368-USB, U18 RK3368_SDMMC, U19 RK3368_HDMI, U2 TLV62565-LibCool, U20 RK3368_SDIO0, U21 SN74LVC1G14DBV, U22 RTL8211E-VB-CG, U23 GL852G, U24 MP65151DJ, U25 GST5009, U26 MP65151DJ, U27 MP65151DJ, U28 AP6335, U29 AT24C16B, U3 TPS72118, U30 RK3368_MAC, U31 MAX3232, U4 TPS62052DGS, U5 MAX1651, U6 TPS7A21, U7 RK3368_ADC, U8 RK3368-USB, U9 RK3368_HSIC, Y1 24MHz, Y2 32.768kHz, Y3 OSC-LibCool, Y4 37.4MHz

Commit message: 5-16 PC
Parts:
- removed AE1: Antenna, symbol Device:Antenna
- removed C1, C79: 4.7uF, symbol Lib1:C(MM)-LibCool
- removed C10, C11, C21, C28, C48, C55: 1uF, symbol Lib1:C(MM)-LibCool
- removed C12, C17, C18, C2, C22, C25, C27, C29, C30, C31, C33, C36, C40, C42, C43, C44, C45, C46, C47, C49, C52, C53, C62, C63, C7, C81, C82, C83, C84: 100nF, symbol Lib1:C(MM)-LibCool
- removed C13, C15, C16, C24, C37, C54: 10nF, symbol Lib1:C(MM)-LibCool
- removed C14, C26, C34, C59: 1nF, symbol Lib1:C(MM)-LibCool
- removed C19, C20: 12pF, symbol Lib1:C(MM)-LibCool
- removed C23, C6: 22uF, symbol Lib1:C(MM)-LibCool
- removed C3: 47uF, symbol Lib1:C(MM)-LibCool
- removed C32, C35, C4, C41, C51, C58, C60, C61, C67, C68: 10uF, symbol Lib1:C(MM)-LibCool
- removed C38, C39, C56, C57, C80: 22pF, symbol Lib1:C(MM)-LibCool
- removed C5, C69, C70: 0.1uF, symbol Lib1:C(MM)-LibCool
- removed C50, C71, C72, C8: 100uF, symbol Lib1:C(MM)-LibCool
- removed C64, C66, C73, C74, C75, C76, C77, C78: 18pF, symbol Lib1:C(MM)-LibCool
- removed C65: 10pF, symbol Lib1:C(MM)-LibCool
- removed C9: 330uF, symbol Lib1:C(MM)-LibCool
- removed D1: SMBJ5.0A, Diode_THT:D_DO-35_SOD27_P7.62mm_Horizontal, symbol Diode:1N6857
- removed D10, D11, D13, D14, D15, D16, D17, D18, D3, D4, D5, D6, D7, D8, D9: ESD9B5VL, Diode_SMD:D_SOD-923, symbol Diode:ESD9B5.0ST5G
- removed D12: PMEG3030BEP, symbol Device:D_Schottky
- removed D2: 1N5820, Diode_THT:D_DO-201AD_P15.24mm_Horizontal, symbol Diode:1N5820
- removed J1: DBG1, symbol Connector:Conn_01x03_Female
- removed J2, J5, J6, J7: USB_A, symbol Connector:USB_A
- removed J3: Micro_SD_Card_Det, symbol Connector:Micro_SD_Card_Det
- removed J4: RJ45, symbol Connector:RJ45
- removed J8: HDMI_A, symbol Connector:HDMI_A
- removed J9: DB9_Male, symbol Connector:DB9_Male
- removed L1: 2.2uH, symbol Lib1:Inductor-LibCool
- removed L2: 10uH, symbol Lib1:Inductor-LibCool
- removed L3: 47uH, symbol Lib1:Inductor-LibCool
- removed L4: 3.3uH, symbol Lib1:Inductor-LibCool
- removed Q1: Si9430, symbol Lib1:PMOS-LibCool
- removed Q2, Q3, Q4: 2N7002, Package_TO_SOT_SMD:SOT-23, symbol Transistor_FET:2N7002
- removed R1, R35: 100K, symbol Lib1:RES(M)-LibCool
- removed R10, R22, R9: 1K, symbol Lib1:RES(M)-LibCool
- removed R100, R101, R102, R103, R104, R105, R93, R94, R95, R96, R97, R98, R99: 22, symbol Lib1:RES(M)-LibCool
- removed R11: 6.8K, symbol Lib1:RES(M)-LibCool
- removed R12, R15, R16, R17, R19, R20, R21, R23, R25, R26, R27, R28, R29, R31, R33, R34, R36, R37, R44, R54, R56, R64, R65, R7, R82: 10K, symbol Lib1:RES(M)-LibCool
- removed R13: 1M, symbol Lib1:RES(M)-LibCool
- removed R14: 510R, symbol Lib1:RES(M)-LibCool
- removed R18, R8: 133R, symbol Lib1:RES(M)-LibCool
- removed R2: 120K, symbol Lib1:RES(M)-LibCool
- removed R24: 1.62K, symbol Lib1:RES(M)-LibCool
- removed R3: 0.05R, symbol Lib1:RES(M)-LibCool
- removed R30, R46, R49, R50, R51, R52, R53, R70, R71, R72, R73, R74, R75: 22R, symbol Lib1:RES(M)-LibCool
- removed R32: 680R, symbol Lib1:RES(M)-LibCool
- removed R38: 2.49K, symbol Lib1:RES(M)-LibCool
- removed R39, R40, R41, R42, R85, R86, R87, R88, R89, R90, R91, R92: 4K7, symbol Lib1:RES(M)-LibCool
- removed R4: 180K, symbol Lib1:RES(M)-LibCool
- removed R43: 1K5, symbol Lib1:RES(M)-LibCool
- removed R45: 15K, symbol Lib1:RES(M)-LibCool
- removed R47, R48, R76, R77, R78, R79, R80, R81: 90, symbol Lib1:RES(M)-LibCool
- removed R5: 150K, symbol Lib1:RES(M)-LibCool
- removed R55, R67, R68: 20K, symbol Lib1:RES(M)-LibCool
- removed R57, R58: 4.7K, symbol Lib1:RES(M)-LibCool
- removed R59, R60, R61, R62: 75, symbol Lib1:RES(M)-LibCool
- removed R6: 100nF, symbol Lib1:RES(M)-LibCool
- removed R63, R66: 1.5K, symbol Lib1:RES(M)-LibCool
- removed R69: 100R, symbol Lib1:RES(M)-LibCool
- removed R83, R84: 2.2K, symbol Lib1:RES(M)-LibCool
- removed TP1, TP2: +5, symbol Connector:TestPoint
- removed TP3: 1V_USB, symbol Connector:TestPoint
- removed TP4: 1V8_USB, symbol Connector:TestPoint
- removed TP5: 3V3_IO, symbol Connector:TestPoint
- removed U1: TPS7A0310, symbol Lib1:TPS7A0310
- removed U10: RK3368_DDR, symbol Lib1:RK3368_DDR
- removed U11: RK3368_SYS, symbol Lib1:RK3368_SYS
- removed U12, U13, U14, U15: MT41KxxxM16TW, Package_BGA:BGA-96_9.0x13.0mm_Layout2x3x16_P0.8mm, symbol Memory_RAM:AS4C256M16D3
- removed U16: RK3368_UART, symbol Lib1:RK3368_UART
- removed U17, U8: RK3368-USB, symbol Lib1:RK3368-USB
- removed U18: RK3368_SDMMC, symbol Lib1:RK3368_SDMMC
- removed U19: RK3368_HDMI, symbol Lib1:RK3368_HDMI
- removed U2: TLV62565-LibCool, symbol Lib1:TLV62565-LibCool
- removed U20: RK3368_SDIO0, symbol Lib1:RK3368_SDIO0
- removed U21: SN74LVC1G14DBV, Package_TO_SOT_SMD:SOT-23-5, symbol 74xGxx:SN74LVC1G14DBV
- removed U22: RTL8211E-VB-CG, symbol Lib1:RTL8211E-VB-CG
- removed U23: GL852G, symbol Lib1:GL852G
- removed U24, U26, U27: MP65151DJ, symbol Lib1:MP65151DJ
- removed U25: GST5009, symbol Lib1:GST5009
- removed U28: AP6335, symbol Lib1:AP6335
- removed U29: AT24C16B, Package_SO:SOIC-8_3.9x4.9mm_P1.27mm, symbol Memory_EEPROM:AT24CS16-SSHM
- removed U3: TPS72118, symbol Lib1:TPS72118
- removed U30: RK3368_MAC, symbol Lib1:RK3368_MAC
- removed U31: MAX3232, symbol Interface_UART:MAX3232
- removed U4: TPS62052DGS, Package_SO:VSSOP-10_3x3mm_P0.5mm, symbol Regulator_Switching:TPS62056DGS
- removed U5: MAX1651, symbol Lib1:MAX1651
- removed U6: TPS7A21, symbol Lib1:TPS7A0310
- removed U7: RK3368_ADC, symbol Lib1:RK3368_ADC
- removed U9: RK3368_HSIC, symbol Lib1:RK3368_HSIC
- removed Y1: 24MHz, symbol Lib1:OSC-LibCool
- removed Y2: 32.768kHz, symbol Lib1:OSC-LibCool
- removed Y3: OSC-LibCool, symbol Lib1:OSC-LibCool
- removed Y4: 37.4MHz, symbol Lib1:OSC-LibCool
- added C1: (no value), symbol Device:C
- added C10, C12, C? (x4): 100nF, symbol Device:C_Small
- added C11, C14, C17, C9: 10nF, symbol Device:C_Small
- added C13: 0.1uF, symbol Device:C_Small
- added C15, C16, C? (x2): 1nF, symbol Device:C_Small
- added C18, C20, C21, C22, C23, C24, C25, C26, C27, C28, C29, C30, C? (x30): (no value), symbol Device:C_Small
- added C19, C8: 1uF, symbol Device:C_Small
- added C2: 4.7uF, symbol Device:C_Small
- added C3, C7: 100uF, symbol Device:C_Small
- added C4: 100uF, symbol Device:C
- added C5: 22uF, symbol Device:C_Polarized_Small
- added C6: 10uF, symbol Device:C_Small
- added C? (x9): 22uF, Capacitor_THT:CP_Radial_D6.3mm_P2.50mm, symbol Device:C_Small
- added C? (x18): 100nF, Capacitor_SMD:C_0603_1608Metric, symbol Device:C_Small
- added C? (x4): 22uF, symbol Device:C_Small
- added C? (x3): 1uF, Capacitor_SMD:C_0603_1608Metric, symbol Device:C_Small
- added D1, D3: MBRS140T3, Diode_THT:D_DO-35_SOD27_P7.62mm_Horizontal, symbol Diode:1N5711
- added D5: LED, symbol Device:LED
- added D6: (no value), symbol Device:LED
- added D? (x2): (no value), symbol Power_Protection:NUP2105L
- added D?: ESD5302F, Package_TO_SOT_SMD:SOT-23, symbol Power_Protection:NUP2105L
- added D?: (no value), symbol Diode:ESD9B5.0ST5G
- added D?: (no value), symbol Diode:BAV70
- added J?: (no value), symbol Connector:USB_C_Receptacle
- added J?: (no value), symbol Connector:USB_A_Stacked
- added J?: (no value), symbol Connector:USB3_A
- added L1, L2: L, symbol Device:L
- added L3, L4, L5: (no value), symbol Device:L
- added Q1, Q2: FDS6890A, Package_SO:SOIC-8_3.9x4.9mm_P1.27mm, symbol Transistor_FET:FDS6890A
- added R1, R13, R14, R15, R16, R17, R18, R19, R2, R20, R21, R4, R5, R? (x7): (no value), symbol Device:R_Small
- added R10, R11: 20K, symbol Device:R_Small
- added R12: 220K, symbol Device:R_Small
- added R3, R7, R9: 4R7, symbol Device:R_Small
- added R6, R8: 13K, symbol Device:R_Small
- added R?: 2M, symbol Device:R_Small
- added R? (x8): 240R, symbol Device:R_Small
- added R?: 133R, symbol Device:R_Small
- added TP? (x2): (no value), symbol Connector:TestPoint
- added U1: CH340E, Package_SO:MSOP-10_3x3mm_P0.5mm, symbol Interface_USB:CH340E
- added U2: (no value), symbol LM2642MTC:LM2642MTC
- added U3: RK3399, BGA828C65P31X31_2100X2100X161N, symbol RK3399:RK3399
- added U4: (no value), symbol MAX15053EWL:MAX15053EWL
- added U5: (no value), symbol Power_Management:MAX1952
- added U6: (no value), Package_TO_SOT_SMD:SOT-23-5, symbol Regulator_Switching:TLV62568DBV
- added U?: (no value), symbol Power_Protection:D3V3XA4B10LP
- added U?: (no value), Package_DFN_QFN:Diodes_UDFN-10_1.0x2.5mm_P0.5mm, symbol Power_Protection:D3V3XA4B10LP
- added U?: ESD5304D, Package_DFN_QFN:Diodes_UDFN-10_1.0x2.5mm_P0.5mm, symbol Power_Protection:D3V3XA4B10LP
- added U?: (no value), symbol FUSB302MPX:FUSB302MPX
- added U? (x3): H5TC4G63AFR, symbol Memory_RAM:H5TC4G63AFR
- added U?: (no value), symbol TPS826745SIPR:TPS826745SIPR
- added U?: (no value), symbol Memory_RAM:H5TC4G63AFR
- added Y?: (no value), symbol Device:Crystal_GND24
- F1: value 5A -> (none)
Connections:
- net +1V5: now also C1.1, C3.2, L1.1, R1.1
- net +1V8: now also C28.1, L4.2, U3.AA18 (TYPEC0_AVDD_1V8), U3.AA21 (TYPEC1_AVDD_1V8), U3.AA8 (APIO5_VDDPST), U3.AB8 (APIO3_VDD_1V8), U3.AC8 (APIO4_VDDPST), U3.AC9 (APIO4_VDD), U3.J22 (APIO1_VDDPST), U3.J23 (APIO1_VDD), U3.J24 (APIO2_VDDPST), U3.K23 (APIO2_VDD)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
- net +3V3: now also C4.1, C7.2, L2.1, R4.1, U3.AB18 (TYPEC0_AVDD_3V3), U3.AB21 (TYPEC1_AVDD_3V3), U3.Y25 (USB_AVDD_3V3), U?.3 (VDD), U?.4 (VDD), U?.A2 (VIN), U?.A3 (VIN), U?.B2 (EN)
- net +5V: now also C11.1, C26.1, C5.1, C6.1, C8.1, C9.1, D?.2 (A2), J?.1 (VBUS1), J?.5 (VBUS2), Q1.7 (D1), Q1.8 (D1), Q2.7 (D1)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
- net A10: now also U3.B10 (DDR1_A0), U?.N3 (A0), U?.N3 (A0)
- net A11: now also U3.A10 (DDR1_A1), U?.P7 (A1), U?.P7 (A1)
- net A12: now also U3.B9 (DDR1_A2), U?.P3 (A2), U?.P3 (A2)
- net A13: now also U3.A9 (DDR1_A3), U?.N2 (A3), U?.N2 (A3)
- net A14: now also U3.B8 (DDR1_A4), U?.P8 (A4), U?.P8 (A4)
- net A15: now also U3.A8 (DDR1_A5), U?.P2 (A5), U?.P2 (A5)
- net GND: now also C1.2, C13.1, C14.1, C17.1, C18.2, C19.2, C2.2, C21.1, C22.1, C23.1, C24.2, C25.2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
- net HOST1_D+: now also D?.2 (K), J?.3 (D1+), U3.AA30 (USB1_DP)
- net HOST1_D-: now also D?.1 (K), J?.2 (D1-), U3.AA31 (USB1_DN)
- net UART1_RX: now also U1.8 (TXD)
- net UART1_TX: now also U1.9 (RXD)
- net at P1.A6 (D+): now also U1.1 (UD+)
- net at P1.A7 (D-): now also U1.2 (UD-)
- new net: D5.2 (A), R12.2, U2.5 (PGOOD1)
- new net: C?.2, C?.2, C?.2, C?.2, C?.2, C?.2, C?.2, C?.2, C?.2, C?.2, C?.2, C?.2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
- new net: C?.1, J?.A2 (TX1+)
- new net: C?.1, J?.A3 (TX1-)
- new net: C?.1, J?.B2 (TX2+)
- new net: C?.1, J?.B3 (TX2-)
- new net: C24.1, R17.1, U5.1 (VCC)
- new net: C27.1, U5.2 (REF)
- new net: R18.2, U5.5 (COMP)
- new net: L4.1, U5.7 (LX)
- new net: R19.2, R20.1, U6.5 (FB)
- new net: C13.2, U2.6 (UVDELAY)
- new net: C22.2, R15.1
- new net: C23.2, R16.1
- new net: R16.2, U4.B1 (COMP)
- new net: R?.1, U?.L9 (ZQ1) (x4)
- new net: C30.1, U4.C2 (SS/REFIN)
- new net: C15.1, R10.2
- new net: C15.2, U2.3 (COMP1)
- new net: C20.1, C21.2, L3.1, R13.1
- new net: C9.2, R6.2, U2.13 (ILIM2)
- new net: L5.1, U6.3 (SW)
- new net: U3.R11 (GPU_VDD_8), U3.R12 (GPU_VDD_9), U3.T11 (GPU_VDD_10), U3.T15 (GPU_VDD_COM), U3.U13 (GPU_VDD_7), U3.V13 (GPU_VDD_6), U3.V14 (GPU_VDD_5), U3.V15 (GPU_VDD_4), U3.W11 (GPU_VDD_1), U3.W12 (GPU_VDD_2), U3.W14 (GPU_VDD_3)
- new net: U3.R13 (GPU_VDD_13), U3.T12 (GPU_VDD_11), U3.T13 (GPU_VDD_12), U3.T14 (GPU_VDD_14), U3.V11 (GPU_VDD_15), U3.V12 (GPU_VDD_16), U3.V16 (GPU_VDD_17), U3.W10 (GPU_VDD_20), U3.W15 (GPU_VDD_19), U3.W16 (GPU_VDD_18)
- new net: U3.P20 (LITCPU_VDD_1), U3.P22 (LITCPU_VDD_4), U3.R19 (LITCPU_VDD_2), U3.R20 (LITCPU_VDD_3)
- new net: U3.R22 (LITCPU_VDD_7), U3.T20 (LITCPU_VDD_6), U3.T22 (LITCPU_VDD_5)
- new net: R?.2, U3.G15 (DDR1_PZQ)
- new net: C11.2, R8.2, U2.2 (ILIM1)
- new net: R?.2, U3.AC31 (USB0_RBIAS)
- new net: D6.2 (A), R21.1, U4.C3 (PGOOD)
- new net: C25.1, R18.1
- new net: R?.1, U?.L8 (ZQ0) (x4)
- new net: C18.1, U1.10 (V3)
- new net: TP?.1, U3.AJ30 (USIC_STROBE)
- new net: C12.2, D?.1 (A), U2.25 (CBOOT1)
- new net: U?.A1 (VDDQ), U?.A8 (VDDQ), U?.C1 (VDDQ), U?.C9 (VDDQ), U?.D2 (VDDQ), U?.E9 (VDDQ), U?.F1 (VDDQ), U?.H2 (VDDQ), U?.H9 (VDDQ)
- new net: U?.B2 (VDD), U?.D9 (VDD), U?.G7 (VDD), U?.K2 (VDD), U?.K8 (VDD), U?.N1 (VDD), U?.N9 (VDD), U?.R1 (VDD), U?.R9 (VDD)
- new net: C14.2, U2.9 (ON/SS1)
- new net: C16.1, R11.2
- new net: L3.2, R15.2, U4.A2 (LX)
- new net: Q1.4 (G2), U2.23 (LDRV1)
- new net: U3.K19 (BIGCPU_VDD_12), U3.K21 (BIGCPU_VDD_13), U3.L18 (BIGCPU_VDD_8), U3.L23 (BIGCPU_VDD_11), U3.N18 (BIGCPU_VDD_COM), U3.N20 (BIGCPU_VDD_10), U3.N22 (BIGCPU_VDD_9)
- new net: U3.L19 (BIGCPU_VDD_1), U3.L21 (BIGCPU_VDD_2), U3.M18 (BIGCPU_VDD_3), U3.M19 (BIGCPU_VDD_4), U3.M20 (BIGCPU_VDD_5), U3.M21 (BIGCPU_VDD_6), U3.M22 (BIGCPU_VDD_7)
- new net: Q2.4 (G2), U2.20 (LDRV2)
- new net: Q1.2 (G1), U2.26 (HDRV1)
- new net: R?.2, U3.R7 (DDR0_PZQ)
- new net: C16.2, U2.12 (COMP2)
- new net: C10.2, D?.2 (A), U2.18 (CBOOT2)
- new net: C17.2, U2.10 (ON/SS2)
- new net: Q2.2 (G1), U2.17 (HDRV2)
- new net: TP?.1, U3.AJ31 (USIC_DATA)
- new net: U3.M11 (CENTERLOGIC_VDD_1), U3.M12 (CENTERLOGIC_VDD_2), U3.M13 (CENTERLOGIC_VDD_3), U3.M14 (CENTERLOGIC_VDD_4), U3.M15 (CENTERLOGIC_VDD_5)
- new net: U3.N11 (CENTERLOGIC_VDD_6), U3.N12 (CENTERLOGIC_VDD_7), U3.P13 (CENTERLOGIC_VDD_8), U3.P14 (CENTERLOGIC_VDD_9), U3.P15 (CENTERLOGIC_VDD_10)
- new net: R?.2, U3.AC30 (USB1_RBIAS)
- new net: U3.AA19 (NC), U3.AA20 (NC), U3.AA22 (NC), U3.AB20 (NC), U3.AB22 (NC), U3.AC12 (NC), U3.AC14 (NC), U3.AD11 (NC), U3.AD12 (NC), U3.AD14 (NC), U3.AD15 (NC)
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Other:
- note removed: "50 Ohm 阻抗控制"
- note removed: "差分布线 50Ohm"

Commit message: 5-17 phone
Parts:
- added R (x2): R_Small, symbol Device:R_Small
- added TP: TestPoint_Alt, symbol Connector:TestPoint_Alt
- added U (x2): (no value), symbol Device:C_Small
- U: renamed from R12; value 220K -> (none)
- U: renamed from R?; value 2M -> (none)
- U: renamed from C?; value 22uF -> (none); footprint Capacitor_THT:CP_Radial_D6.3mm_P2.50mm -> (none)
- U: renamed from C?; value 100nF -> (none); footprint Capacitor_SMD:C_0603_1608Metric -> (none)
- U: renamed from U?; footprint Package_DFN_QFN:Diodes_UDFN-10_1.0x2.5mm_P0.5mm -> (none)
- U: renamed from U?; value ESD5304D -> (none); footprint Package_DFN_QFN:Diodes_UDFN-10_1.0x2.5mm_P0.5mm -> (none)
- U: renamed from C?; value 1nF -> (none)
- U: renamed from C?; value 100nF -> (none)
- U: renamed from C13; value 0.1uF -> (none)
- U: renamed from U3; value RK3399 -> (none); footprint BGA828C65P31X31_2100X2100X161N -> (none)
- U: renamed from D3; value MBRS140T3 -> (none); footprint Diode_THT:D_DO-35_SOD27_P7.62mm_Horizontal -> (none)
- U: renamed from R?; value 240R -> (none)
- U: renamed from C?; value 22uF -> (none)
- U: renamed from C15; value 1nF -> (none)
- U: renamed from R6; value 13K -> (none)
- U: renamed from C4; value 100uF -> (none)
- U: renamed from C?; value 1uF -> (none); footprint Capacitor_SMD:C_0603_1608Metric -> (none)
- U: renamed from R8; value 13K -> (none)
- U: renamed from L2; value L -> (none)
- U: renamed from D?; value ESD5302F -> (none); footprint Package_TO_SOT_SMD:SOT-23 -> (none)
- U: renamed from L1; value L -> (none)
- U: renamed from U?; value H5TC4G63AFR -> (none)
- U: renamed from R9; value 4R7 -> (none)
- U: renamed from C12; value 100nF -> (none)
- U: renamed from C14; value 10nF -> (none)
- U: renamed from R11; value 20K -> (none)
- U: renamed from C3; value 100uF -> (none)
- U: renamed from Q1; value FDS6890A -> (none); footprint Package_SO:SOIC-8_3.9x4.9mm_P1.27mm -> (none)
- U: renamed from D1; value MBRS140T3 -> (none); footprint Diode_THT:D_DO-35_SOD27_P7.62mm_Horizontal -> (none)
- U: renamed from C2; value 4.7uF -> (none)
- U: renamed from C11; value 10nF -> (none)
- U: renamed from Q2; value FDS6890A -> (none); footprint Package_SO:SOIC-8_3.9x4.9mm_P1.27mm -> (none)
- U: renamed from C9; value 10nF -> (none)
- U: renamed from C7; value 100uF -> (none)
- U: renamed from C16; value 1nF -> (none)
- U: renamed from C10; value 100nF -> (none)
- U: renamed from C6; value 10uF -> (none)
- U: renamed from C8; value 1uF -> (none)
- U: renamed from C5; value 22uF -> (none)
- U: renamed from R3; value 4R7 -> (none)
- U: renamed from C17; value 10nF -> (none)
- U: renamed from P1; value USB_C_Plug_USB2.0 -> (none)
- U: renamed from R10; value 20K -> (none)
- U: renamed from R7; value 4R7 -> (none)
- U: renamed from U1; value CH340E -> (none); footprint Package_SO:MSOP-10_3x3mm_P0.5mm -> (none)
- U: renamed from D5; value LED -> (none)
- U: renamed from R?; value 133R -> (none)
- U: renamed from C19; value 1uF -> (none)
- U: renamed from U6; footprint Package_TO_SOT_SMD:SOT-23-5 -> (none)
- gave numbers to parts that had none: 7
- renumbered R17 to U, U5 to U, R20 to U, C22 to U, C24 to U, R16 to U, C30 to U, L4 to U, C21 to U, L5 to U, C27 to U, D6 to U, R18 to U, R1 to U, C28 to U, C18 to U, C23 to U, C29 to U, R15 to U, R21 to U, R13 to U, C26 to U, R14 to U, C25 to U, L3 to U, F1 to U, C20 to U, U2 to U, C1 to U, U4 to U, R4 to U, R5 to U, R2 to U, R19 to U
Connections:
- net +0V9: no longer U.AD25 (USIC_AVDD_0V9), U.V24 (USB_AVDD_0V9), U.Y18 (TYPEC0_AVDD_0V9_2), U.Y19 (TYPEC0_AVDD_0V9_1), U.Y21 (TYPEC1_AVDD_0V9_1), U.Y22 (TYPEC1_AVDD_0V9_2)
- net +1V2: no longer U.AD24 (USIC_AVDD_1V2)
- net +1V8: no longer U.AA18 (TYPEC0_AVDD_1V8), U.AA21 (TYPEC1_AVDD_1V8), U.AA8 (APIO5_VDDPST), U.AB8 (APIO3_VDD_1V8), U.AC8 (APIO4_VDDPST), U.AC9 (APIO4_VDD), U.J22 (APIO1_VDDPST), U.J23 (APIO1_VDD), U.J24 (APIO2_VDDPST), U.K23 (APIO2_VDD), U.N23 (PMUIO2_VDDPST), U.P18 (PLL_AVDD_1V8)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
- net +3V0: no longer U.P23 (PMUIO2_VDD)
- net +3V3: no longer U.AB18 (TYPEC0_AVDD_3V3), U.AB21 (TYPEC1_AVDD_3V3), U.Y25 (USB_AVDD_3V3)
- net 0CASN: now also U.P10 (VSS_116); no longer U.H6 (DDR0_CASN)
- net 0CKE0: now also U.W30 (VSS_160); no longer U.E1 (DDR0_CKE0)
- net 0CKE1: now also U.W8 (VSS_161); no longer U.F5 (DDR0_CKE1)
- net 0CS0: now also U.R3 (VSS_123); no longer U.M6 (DDR0_CSN0)
- net 0CS1: now also U.R5 (VSS_124); no longer U.B1 (DDR0_CSN1)
- net 0D0: now also U.AD5 (VSS_18); no longer U.AB2 (DDR0_DQ0)
- net 0D1: now also U.AD10 (VSS_19); no longer U.AB1 (DDR0_DQ1)
- net 0D10: now also U.C12 (VSS_28); no longer U.AF1 (DDR0_DQ10)
- net 0D11: now also U.C14 (VSS_29); no longer U.AD2 (DDR0_DQ11)
- net 0D12: now also U.C15 (VSS_30); no longer U.AE1 (DDR0_DQ12)
- net 0D13: now also U.C17 (VSS_31); no longer U.AD1 (DDR0_DQ13)
- net 0D14: now also U.C18 (VSS_32); no longer U.AC1 (DDR0_DQ14)
- net 0D15: now also U.C20 (VSS_33); no longer U.AC2 (DDR0_DQ15)
- net 0D16: now also U.C21 (VSS_34); no longer U.V1 (DDR0_DQ16)
- net 0D17: now also U.C23 (VSS_35); no longer U.V2 (DDR0_DQ17)
- net 0D18: now also U.C24 (VSS_36); no longer U.U1 (DDR0_DQ18)
- net 0D19: now also U.C26 (VSS_37); no longer U.U2 (DDR0_DQ19)
- net 0D2: now also U.AF9 (VSS_20); no longer U.AA2 (DDR0_DQ2)
- net 0D20: now also U.D5 (VSS_38); no longer U.T1 (DDR0_DQ20)
- net 0D21: now also U.E2 (VSS_39); no longer U.T2 (DDR0_DQ21)
- net 0D22: now also U.E4 (VSS_40); no longer U.R2 (DDR0_DQ22)
- net 0D23: now also U.E7 (VSS_41); no longer U.R1 (DDR0_DQ23)
- net 0D24: now also U.E12 (VSS_42); no longer U.P1 (DDR0_DQ24)
- net 0D25: now also U.E15 (VSS_43); no longer U.P2 (DDR0_DQ25)
- net 0D26: now also U.E18 (VSS_44); no longer U.N1 (DDR0_DQ26)
- net 0D27: now also U.E21 (VSS_45); no longer U.M1 (DDR0_DQ27)
- net 0D28: now also U.E24 (VSS_46); no longer U.N2 (DDR0_DQ28)
- net 0D29: now also U.E31 (VSS_47); no longer U.L1 (DDR0_DQ29)
- net 0D3: now also U.AG2 (VSS_21); no longer U.AA1 (DDR0_DQ3)
- net 0D30: now also U.F8 (VSS_48); no longer U.M2 (DDR0_DQ30)
- net 0D31: now also U.F15 (VSS_49); no longer U.L2 (DDR0_DQ31)
- net 0D4: now also U.AJ5 (VSS_22); no longer U.Y2 (DDR0_DQ4)
- net 0D5: now also U.AL1 (VSS_23); no longer U.Y1 (DDR0_DQ5)
- net 0D6: now also U.B5 (VSS_24); no longer U.W1 (DDR0_DQ6)
- net 0D7: now also U.C8 (VSS_25); no longer U.W2 (DDR0_DQ7)
- net 0D8: now also U.C9 (VSS_26); no longer U.AF2 (DDR0_DQ8)
- net 0D9: now also U.C11 (VSS_27); no longer U.AE2 (DDR0_DQ9)
- new net: U.A1 (VSS_1), U.AD3 (VSS_17), U.C15 (VSS_30)
- new net: U.A27 (VSS_2), U.AD5 (VSS_18), U.C17 (VSS_31)
- new net: U.A31 (VSS_3), U.AD10 (VSS_19), U.C18 (VSS_32)
- new net: U.AA3 (VSS_4), U.AF9 (VSS_20), U.C20 (VSS_33)
- new net: U.AA5 (VSS_5), U.AG2 (VSS_21), U.C21 (VSS_34)
- new net: U.AA9 (VSS_6), U.AJ5 (VSS_22), U.C23 (VSS_35)
- new net: U.AB19 (VSS_140), U.W18 (VSS_169), U.Y14 (VSS_156)
- new net: U.AB9 (VSS_9), U.C8 (VSS_25), U.D5 (VSS_38)
- new net: U.AC18 (VSS_145), U.AJ24 (VSS_174), U.W8 (VSS_161)
- new net: U.AC20 (VSS_13), U.C14 (VSS_29), U.E12 (VSS_42)
- new net: U.AC21 (VSS_132), U.V17 (VSS_148), U.W8 (VSS_161)
- new net: U.AC22 (VSS_12), U.C12 (VSS_28), U.E7 (VSS_41)
- new net: U.AC3 (VSS_16), U.C18 (VSS_32), U.E21 (VSS_45)
- new net: U.AD10 (VSS_19), U.C23 (VSS_35), U.F8 (VSS_48)
- new net: U.AA10 (VSS_179), U.AD21 (VSS_163)
- new net: U.AD22 (VSS_11), U.C11 (VSS_27), U.E4 (VSS_40)
- new net: U.AD3 (VSS_17), U.C20 (VSS_33), U.E24 (VSS_46)
- new net: U.AD5 (VSS_18), U.C21 (VSS_34), U.E31 (VSS_47)
- new net: U.AE23 (VSS_14), U.C15 (VSS_30), U.E15 (VSS_43)
- new net: U.AF18 (VSS_7), U.AL1 (VSS_23), U.C24 (VSS_36)
- new net: U.AF20 (VSS_10), U.C9 (VSS_26), U.E2 (VSS_39)
- new net: U.AF9 (VSS_20), U.C24 (VSS_36), U.F15 (VSS_49)
- new net: U.AG2 (VSS_21), U.C26 (VSS_37), U.F18 (VSS_50)
- new net: U.AJ5 (VSS_22), U.D5 (VSS_38), U.F20 (VSS_51)
- new net: U.AL1 (VSS_23), U.E2 (VSS_39), U.F21 (VSS_52)
- new net: U.B5 (VSS_24), U.E4 (VSS_40), U.G5 (VSS_53)
- new net: U.C11 (VSS_27), U.E15 (VSS_43), U.G27 (VSS_56)
- new net: U.C12 (VSS_28), U.E18 (VSS_44), U.H3 (VSS_57)
- new net: U.C14 (VSS_29), U.E21 (VSS_45), U.H9 (VSS_58)
- new net: U.C15 (VSS_30), U.E24 (VSS_46), U.H10 (VSS_59)
- new net: U.C17 (VSS_31), U.E31 (VSS_47), U.H11 (VSS_60)
- new net: U.C18 (VSS_32), U.F8 (VSS_48), U.H12 (VSS_61)
- new net: U.C20 (VSS_33), U.F15 (VSS_49), U.H13 (VSS_62)
- new net: U.C21 (VSS_34), U.F18 (VSS_50), U.H15 (VSS_63)
- new net: U.C23 (VSS_35), U.F20 (VSS_51), U.H16 (VSS_64)
- new net: U.C24 (VSS_36), U.F21 (VSS_52), U.H17 (VSS_65)
- new net: U.C26 (VSS_37), U.G5 (VSS_53), U.H18 (VSS_66)
- new net: U.C8 (VSS_25), U.E7 (VSS_41), U.G9 (VSS_54)
- new net: U.C9 (VSS_26), U.E12 (VSS_42), U.G18 (VSS_55)
- new net: U.D5 (VSS_38), U.G9 (VSS_54), U.H26 (VSS_67)
- new net: U.E12 (VSS_42), U.H9 (VSS_58), U.J8 (VSS_71)
- new net: U.E15 (VSS_43), U.H10 (VSS_59), U.J9 (VSS_72)
- new net: U.E18 (VSS_44), U.H11 (VSS_60), U.J10 (VSS_73)
- new net: U.E2 (VSS_39), U.G18 (VSS_55), U.J3 (VSS_68)
- new net: U.E21 (VSS_45), U.H12 (VSS_61), U.K8 (VSS_74)
- new net: U.E24 (VSS_46), U.H13 (VSS_62), U.K9 (VSS_75)
- new net: U.E31 (VSS_47), U.H15 (VSS_63), U.K10 (VSS_76)
- new net: U.E4 (VSS_40), U.G27 (VSS_56), U.J6 (VSS_69)
- new net: U.E7 (VSS_41), U.H3 (VSS_57), U.J7 (VSS_70)
- new net: U.F15 (VSS_49), U.H17 (VSS_65), U.K14 (VSS_78)
- new net: U.F18 (VSS_50), U.H18 (VSS_66), U.K16 (VSS_79)
- new net: U.F20 (VSS_51), U.H26 (VSS_67), U.K18 (VSS_80)
- new net: U.F21 (VSS_52), U.J3 (VSS_68), U.W21 (VSS_81)
- new net: U.F8 (VSS_48), U.H16 (VSS_64), U.K12 (VSS_77)
- new net: U.G18 (VSS_55), U.J8 (VSS_71), U.K22 (VSS_84)
- new net: U.G27 (VSS_56), U.J9 (VSS_72), U.L3 (VSS_85)
- new net: U.G5 (VSS_53), U.J6 (VSS_69), U.K20 (VSS_82)
- new net: U.G9 (VSS_54), U.J7 (VSS_70), U.N19 (VSS_83)
- new net: U.H10 (VSS_59), U.K9 (VSS_75), U.L11 (VSS_88)
- new net: U.H11 (VSS_60), U.K10 (VSS_76), U.L12 (VSS_89)
- new net: U.H12 (VSS_61), U.K12 (VSS_77), U.L13 (VSS_90)
- new net: U.H13 (VSS_62), U.K14 (VSS_78)
- new net: U.H15 (VSS_63), U.K16 (VSS_79)
- new net: U.H16 (VSS_64), U.K18 (VSS_80)
- new net: U.H17 (VSS_65), U.W21 (VSS_81)
- new net: U.H18 (VSS_66), U.K20 (VSS_82)
- new net: U.H26 (VSS_67), U.N19 (VSS_83)
- new net: U.H3 (VSS_57), U.J10 (VSS_73), U.L6 (VSS_86)
- new net: U.H9 (VSS_58), U.K8 (VSS_74), U.L8 (VSS_87)
- new net: U.J10 (VSS_73), U.L12 (VSS_89)
- new net: U.J3 (VSS_68), U.K22 (VSS_84)
- new net: U.J6 (VSS_69), U.L3 (VSS_85)
- new net: U.J7 (VSS_70), U.L6 (VSS_86)
- new net: U.J8 (VSS_71), U.L8 (VSS_87)
- new net: U.J9 (VSS_72), U.L11 (VSS_88)
- new net: U.K8 (VSS_74), U.L13 (VSS_90)
- new net: U.L14 (VSS_91), U.P12 (VSS_107), U.R21 (VSS_120)
- new net: U.L15 (VSS_92), U.N13 (VSS_108), U.P21 (VSS_121)
- new net: U.L16 (VSS_93), U.N14 (VSS_109), U.T19 (VSS_122)
- new net: U.L20 (VSS_96), U.P3 (VSS_112), U.R6 (VSS_125)
- new net: U.L22 (VSS_97), U.P6 (VSS_113), U.U11 (VSS_126)
- new net: U.L27 (VSS_99), U.P8 (VSS_115), U.W13 (VSS_128)
- new net: U.M10 (VSS_102), U.R16 (VSS_131), U.Y16 (VSS_118)
- new net: U.AC21 (VSS_132), U.M16 (VSS_103), U.P19 (VSS_119)
- new net: U.M23 (VSS_104), U.R21 (VSS_120), U.R23 (VSS_133)
- new net: U.M3 (VSS_100), U.P10 (VSS_116), U.R14 (VSS_129)
- new net: U.M8 (VSS_101), U.P16 (VSS_117), U.R15 (VSS_130)
- new net: U.N13 (VSS_108), U.R5 (VSS_124), U.U14 (VSS_137)
- new net: U.N14 (VSS_109), U.R6 (VSS_125), U.T16 (VSS_138)
- new net: U.N15 (VSS_110), U.T21 (VSS_139), U.U11 (VSS_126)
- new net: U.AB19 (VSS_140), U.N16 (VSS_111), U.U12 (VSS_127)
- new net: U.N15 (VSS_110), U.N17 (VSS_94), U.R3 (VSS_123)
- new net: U.N21 (VSS_98), U.P7 (VSS_114), U.U12 (VSS_127)
- new net: U.N8 (VSS_105), U.P21 (VSS_121), U.T8 (VSS_134)
- new net: U.AC18 (VSS_145), U.AC21 (VSS_132), U.P10 (VSS_116)
- new net: U.P11 (VSS_106), U.T10 (VSS_135), U.T19 (VSS_122)
- new net: U.P12 (VSS_107), U.R3 (VSS_123), U.Y12 (VSS_136)
- new net: U.P16 (VSS_117), U.R23 (VSS_133), U.U19 (VSS_146)
- new net: U.P19 (VSS_119), U.T10 (VSS_135), U.V17 (VSS_148)
- new net: U.P21 (VSS_121), U.U14 (VSS_137), U.U29 (VSS_150)
- new net: U.P3 (VSS_112), U.U3 (VSS_141), U.W13 (VSS_128)
- new net: U.P6 (VSS_113), U.R14 (VSS_129), U.U8 (VSS_142)
- new net: U.P7 (VSS_114), U.R15 (VSS_130), U.U15 (VSS_143)
- new net: U.P8 (VSS_115), U.R16 (VSS_131), U.U16 (VSS_144)
- new net: U.AC18 (VSS_145), U.R14 (VSS_129), U.W22 (VSS_158)
- new net: U.R15 (VSS_130), U.U19 (VSS_146), U.W17 (VSS_159)
- new net: U.R16 (VSS_131), U.U21 (VSS_147), U.W30 (VSS_160)
- new net: U.R21 (VSS_120), U.U22 (VSS_149), U.Y12 (VSS_136)
- new net: U.R23 (VSS_133), U.U22 (VSS_149), U.W9 (VSS_162)
- new net: U.R3 (VSS_123), U.T21 (VSS_139), U.V5 (VSS_152)
- new net: U.AB19 (VSS_140), U.R5 (VSS_124), U.V8 (VSS_153)
- new net: U.R6 (VSS_125), U.U3 (VSS_141), U.V10 (VSS_154)
- new net: U.T10 (VSS_135), U.V3 (VSS_151), U.Y13 (VSS_164)
- new net: U.T16 (VSS_138), U.V10 (VSS_154), U.W19 (VSS_167)
- new net: U.T16 (VSS_138), U.T19 (VSS_122), U.V3 (VSS_151)
- new net: U.T18 (VSS_168), U.T21 (VSS_139), U.Y11 (VSS_155)
- new net: U.AD21 (VSS_163), U.T8 (VSS_134), U.U29 (VSS_150)
- new net: U.U11 (VSS_126), U.U8 (VSS_142), U.Y11 (VSS_155)
- new net: U.U12 (VSS_127), U.U15 (VSS_143), U.Y14 (VSS_156)
- new net: U.U14 (VSS_137), U.V8 (VSS_153), U.Y9 (VSS_166)
- new net: U.AJ21 (VSS_172), U.U15 (VSS_143), U.W17 (VSS_159)
- new net: U.AJ23 (VSS_173), U.U16 (VSS_144), U.W30 (VSS_160)
- new net: U.AJ26 (VSS_175), U.U19 (VSS_146), U.W9 (VSS_162)
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Other:
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
Commit message: 原理图完工
Parts:
- added AE: Antenna, symbol Device:Antenna
- added C (x28): C_Small, symbol Device:C_Small
- added D (x15): ESD9B3.3ST5G, Diode_SMD:D_SOD-923, symbol Diode:ESD9B3.3ST5G
- added D: LED, symbol Device:LED
- added D (x2): 1N5819, Diode_THT:D_DO-41_SOD81_P10.16mm_Horizontal, symbol Diode:1N5819
- added D: BZT52Bxx, Diode_SMD:D_SOD-123F, symbol Diode:BZT52Bxx
- added J (x3): Conn_01x05_Male, symbol Connector:Conn_01x05_Male
- added J (x2): Conn_01x04_Male, symbol Connector:Conn_01x04_Male
- added J: HR911130A, HANRUN_HR911130A, symbol HR911130A:HR911130A
- added J: Conn_01x14_Male, symbol Connector:Conn_01x14_Male
- added J: Micro_SD_Card_Det, symbol Connector:Micro_SD_Card_Det
- added J: Conn_01x06_Male, symbol Connector:Conn_01x06_Male
- added J: HDMI_A, symbol Connector:HDMI_A
- added L (x3): L, symbol Device:L
- added Q (x3): Q_NMOS_GSD, symbol Device:Q_NMOS_GSD
- added Q: S8050, Package_TO_SOT_THT:TO-92_Inline, symbol Transistor_BJT:S8050
- added R (x58): R_Small, symbol Device:R_Small
- added TP: TestPoint, symbol Connector:TestPoint
- added U: RTL8211D-VB-GR, QFN40P600X600X100-49N, symbol RTL8211D-VB-GR:RTL8211D-VB-GR
- added U: PT5108E23E-30, symbol Power_Management:PT5108E23E-30
- added U: KLMAG2GEND-B031, BGA153N50P14X14_1150X1300X80N, symbol KLMAG2GEND-B031:KLMAG2GEND-B031
- added U: AP6335, symbol AP6335:AP6335
- added X (x2): SG-210SCD, Oscillator:Oscillator_SMD_SeikoEpson_SG210-4Pin_2.5x2.0mm, symbol Oscillator:SG-210SCD
- added Y (x2): Crystal_GND24_Small, symbol Device:Crystal_GND24_Small
Connections:
- net VBus_C is gone; now on net +5V: U.2 (VBUS), U.A4 (VBUS), U.A9 (VBUS), U.B4 (VBUS), U.B9 (VBUS)
- net +0V9: now also U.AB19 (VSS_140), U.AC20 (VSS_13), U.AC21 (VSS_132), U.AD10 (VSS_19), U.AD3 (VSS_17), U.AG2 (VSS_21), U.AJ21 (VSS_172), U.AJ23 (VSS_173), U.AJ24 (VSS_174), U.AJ26 (VSS_175), U.AJ28 (VSS_171), U.AL1 (VSS_23)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
- net +1V8: now also U.R14 (VSS_129), C.2, R.1, R.2, R.2, R.2, R.2, R.2, R.2, R.2, R.2, R.2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
- net +3V0: now also R.2, R.2, U.1, U.1, U.1, U.1, U.1, U.1, U.1, U.1, U.1, U.1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
- net +3V3: now also C.1, C.2, D.2 (A), D.2 (A), D.2 (A), L.1, R.1, U.1 (IN), U.15 (DVDD33), U.21 (DVDD33), U.22 (VDDIO), U.37 (DVDD33)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
- net WIFI_REG_ON_H: now also U.12 (WL_REG_ON)
- net PCIE_TX3+: now reaches U.AB19 (VSS_140)
- net PCIE_TX0-: now reaches U.AC21 (VSS_132)
- net PCIE_RX0+: now reaches U.D5 (VSS_38)
- net PCIE_RX1-: now reaches U.E12 (VSS_42)
- net PCIE_RX2+: now reaches U.E18 (VSS_44)
- net PCIE_RX0-: now reaches U.E2 (VSS_39)
- net PCIE_RX2-: now reaches U.E21 (VSS_45)
- net PCIE_RX3+: now reaches U.E31 (VSS_47)
- net PCIE_RX1+: now reaches U.E7 (VSS_41)
- net PCIE_CLKREQ: now reaches U.F18 (VSS_50)
- net PCIE_RX3-: now reaches U.F8 (VSS_48)
- net PCIE_TX0+: now reaches U.R16 (VSS_131)
- net PCIE_TX1-: now reaches U.T10 (VSS_135)
- net PCIE_TX2-: now reaches U.T16 (VSS_138)
- net PCIE_TX1+: now reaches U.T8 (VSS_134)
- net PCIE_TX2+: now reaches U.U14 (VSS_137)
- net PCIE_REF-: now reaches U.U15 (VSS_143)
- net PCIE_REF+: now reaches U.U16 (VSS_144)
- net PCIE_TX3-: now reaches U.U3 (VSS_141)
- net SDIO_D2: now reaches U.L14 (VSS_91)
- net SDIO_D2: now also R.1
- net SDIO_D3: now reaches U.L15 (VSS_92)
- net SDIO_D3: now also R.1
- net WIFI_HOST_WAKE_L: now reaches U.L16 (VSS_93)
- net WIFI_HOST_WAKE_L: now also U.13 (WL_HOST_WAKE)
- net SDIO_CMD: now reaches U.N17 (VSS_94)
- net SDIO_CMD: now also R.1
- net at U.A1 (VSS_1), U.AD5 (VSS_18): no longer U.E18 (VSS_44)
- net at U.A27 (VSS_2), U.AD10 (VSS_19): no longer U.E21 (VSS_45)
- net at U.A31 (VSS_3), U.AF9 (VSS_20): no longer U.E24 (VSS_46)
- net at U.AA3 (VSS_4), U.AG2 (VSS_21): no longer U.E31 (VSS_47)
- net at U.AA5 (VSS_5), U.AJ5 (VSS_22): no longer U.F8 (VSS_48)
- net at U.AA9 (VSS_6), U.AL1 (VSS_23): no longer U.F15 (VSS_49)
- net at U.AB9 (VSS_9), U.C9 (VSS_26): no longer U.F21 (VSS_52)
- net at U.AC20 (VSS_13), U.C15 (VSS_30): no longer U.G27 (VSS_56)
- net at U.AC21 (VSS_132), U.U22 (VSS_149): no longer U.AJ26 (VSS_175)
- net at U.AC22 (VSS_12), U.C14 (VSS_29): no longer U.G18 (VSS_55)
- net at U.AC3 (VSS_16), U.C20 (VSS_33): no longer U.H10 (VSS_59)
- net at U.AD10 (VSS_19), U.C24 (VSS_36): no longer U.H13 (VSS_62)
- net at U.AD22 (VSS_11), U.C12 (VSS_28): no longer U.G9 (VSS_54)
- net at U.AD3 (VSS_17), U.C21 (VSS_34): no longer U.H11 (VSS_60)
- net at U.AD5 (VSS_18), U.C23 (VSS_35): no longer U.H12 (VSS_61)
- net at U.AE23 (VSS_14), U.C17 (VSS_31): no longer U.H3 (VSS_57)
- net at U.AF18 (VSS_7), U.B5 (VSS_24): no longer U.F18 (VSS_50)
- net at U.AF20 (VSS_10), U.C11 (VSS_27): no longer U.G5 (VSS_53)
- net at U.AF9 (VSS_20), U.C26 (VSS_37): no longer U.H15 (VSS_63)
- net at U.AG2 (VSS_21), U.D5 (VSS_38): no longer U.H16 (VSS_64)
- net at U.AJ5 (VSS_22), U.E2 (VSS_39): no longer U.H17 (VSS_65)
- net at U.AL1 (VSS_23), U.E4 (VSS_40): no longer U.H18 (VSS_66)
- net at U.B5 (VSS_24), U.E7 (VSS_41): no longer U.H26 (VSS_67)
- net at U.C11 (VSS_27), U.E18 (VSS_44): no longer U.J7 (VSS_70)
- net at U.C12 (VSS_28), U.E21 (VSS_45): no longer U.J8 (VSS_71)
- net at U.C14 (VSS_29), U.E24 (VSS_46): no longer U.J9 (VSS_72)
- net at U.C15 (VSS_30), U.E31 (VSS_47): no longer U.J10 (VSS_73)
- net at U.C17 (VSS_31), U.F8 (VSS_48): no longer U.K8 (VSS_74)
- net at U.C18 (VSS_32), U.F15 (VSS_49): no longer U.K9 (VSS_75)
- net at U.C20 (VSS_33), U.F18 (VSS_50): no longer U.K10 (VSS_76)
- net at U.C21 (VSS_34), U.F20 (VSS_51): no longer U.K12 (VSS_77)
- net at U.C23 (VSS_35), U.F21 (VSS_52): no longer U.K14 (VSS_78)
- net at U.C24 (VSS_36), U.G5 (VSS_53): no longer U.K16 (VSS_79)
- net at U.C26 (VSS_37), U.G9 (VSS_54): no longer U.K18 (VSS_80)
- net at U.C8 (VSS_25), U.E12 (VSS_42): no longer U.J3 (VSS_68)
- net at U.C9 (VSS_26), U.E15 (VSS_43): no longer U.J6 (VSS_69)
- net at U.D5 (VSS_38), U.G18 (VSS_55): no longer U.W21 (VSS_81)
- net at U.E12 (VSS_42), U.H10 (VSS_59): no longer U.L3 (VSS_85)
- net at U.E15 (VSS_43), U.H11 (VSS_60): no longer U.L6 (VSS_86)
- net at U.E18 (VSS_44), U.H12 (VSS_61): no longer U.L8 (VSS_87)
- net at U.E2 (VSS_39), U.G27 (VSS_56): no longer U.K20 (VSS_82)
- net at U.E21 (VSS_45), U.H13 (VSS_62): no longer U.L11 (VSS_88)
- net at U.E24 (VSS_46), U.H15 (VSS_63): no longer U.L12 (VSS_89)
- net at U.E31 (VSS_47), U.H16 (VSS_64): no longer U.L13 (VSS_90)
- net at U.E4 (VSS_40), U.H3 (VSS_57): no longer U.N19 (VSS_83)
- net at U.E7 (VSS_41), U.H9 (VSS_58): no longer U.K22 (VSS_84)
- net at U.L14 (VSS_91), U.N13 (VSS_108): no longer U.T8 (VSS_134)
- net at U.L15 (VSS_92), U.N14 (VSS_109): no longer U.T10 (VSS_135)
- net at U.L16 (VSS_93), U.N15 (VSS_110): no longer U.Y12 (VSS_136)
- net at U.L20 (VSS_96), U.P6 (VSS_113): no longer U.T21 (VSS_139)
- net at U.L22 (VSS_97), U.P7 (VSS_114): no longer U.AB19 (VSS_140)
- net at U.L27 (VSS_99), U.P10 (VSS_116): no longer U.U8 (VSS_142)
- net at U.M10 (VSS_102), U.P19 (VSS_119): no longer U.AC18 (VSS_145)
- net at U.M16 (VSS_103), U.R21 (VSS_120): no longer U.U19 (VSS_146)
- net at U.M23 (VSS_104), U.P21 (VSS_121): no longer U.U21 (VSS_147)
- net at U.M3 (VSS_100), U.P16 (VSS_117): no longer U.U15 (VSS_143)
- net at U.M8 (VSS_101), U.Y16 (VSS_118): no longer U.U16 (VSS_144)
- net at U.N13 (VSS_108), U.R6 (VSS_125): no longer U.V3 (VSS_151)
- net at U.N14 (VSS_109), U.U11 (VSS_126): no longer U.V5 (VSS_152)
- net at U.N15 (VSS_110), U.U12 (VSS_127): no longer U.V8 (VSS_153)
- net at U.N16 (VSS_111), U.W13 (VSS_128): no longer U.V10 (VSS_154)
- net at U.N16 (VSS_111), U.N17 (VSS_94): no longer U.U14 (VSS_137)
- net at U.N21 (VSS_98), U.P8 (VSS_115): no longer U.U3 (VSS_141)
- net at U.N8 (VSS_105), U.T19 (VSS_122): no longer U.V17 (VSS_148)
- net at U.P10 (VSS_116), U.R23 (VSS_133): no longer U.W17 (VSS_159)
- net at U.P11 (VSS_106), U.R3 (VSS_123): no longer U.U22 (VSS_149)
- net at U.P12 (VSS_107), U.R5 (VSS_124): no longer U.U29 (VSS_150)
- net at U.P16 (VSS_117), U.T8 (VSS_134): no longer U.W30 (VSS_160)
- net at U.P19 (VSS_119), U.Y12 (VSS_136): no longer U.W9 (VSS_162)
- net at U.P21 (VSS_121), U.T16 (VSS_138): no longer U.Y13 (VSS_164)
- net at U.P3 (VSS_112), U.R14 (VSS_129): no longer U.Y11 (VSS_155)
- net at U.P6 (VSS_113), U.R15 (VSS_130): no longer U.Y14 (VSS_156)
- net at U.P7 (VSS_114), U.R16 (VSS_131): no longer U.Y15 (VSS_157)
- net at U.AC21 (VSS_132), U.P8 (VSS_115): no longer U.W22 (VSS_158)
- net at U.R14 (VSS_129), U.U19 (VSS_146): no longer U.AJ21 (VSS_172)
- net at U.R15 (VSS_130), U.U21 (VSS_147): no longer U.AJ23 (VSS_173)
- net at U.R16 (VSS_131), U.V17 (VSS_148): no longer U.AJ24 (VSS_174)
- net at U.R21 (VSS_120), U.U14 (VSS_137): no longer U.AD21 (VSS_163)
- net at U.R23 (VSS_133), U.U29 (VSS_150): no longer U.AJ27 (VSS_176)
- net at U.AB19 (VSS_140), U.R3 (VSS_123): no longer U.Y9 (VSS_166)
- net at U.R5 (VSS_124), U.U3 (VSS_141): no longer U.W19 (VSS_167)
- net at U.R6 (VSS_125), U.U8 (VSS_142): no longer U.T18 (VSS_168)
- net at U.T10 (VSS_135), U.V5 (VSS_152): no longer U.AL31 (VSS_178)
- net at U.T19 (VSS_122), U.T21 (VSS_139): no longer U.R18 (VSS_165)
- removed net GND: R.2, R.2, U.1, U.1, U.1, U.1, U.1, U.1, U.1, U.1, U.1, U.1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
- new net: Q.2 (B), R.1, R.2
- new net: C.2, U.29 (PHYRSTB)
- new net: U.42 (CKXTAL1), Y.1
- new net: U.43 (CKXTAL2), Y.3
- new net: L.1, U.48 (REG_OUT)
- new net: C.2, U.10 (XTAL_IN), Y.3
- new net: D.2 (A2), J.7 (DAT0), R.2
- new net: C.1, C.1, C.1, C.1, C.1, C.1, C.1, C.1, L.2
- new net: D.1 (K), R.1 (x2)
- new net: Q.3 (C), R.2
- new net: R.2, U.3 (EN)
- new net: C.1, U.4 (BP)
- new net: C.2, R.2, U.18 (SDIO_DATA_0)
- new net: D.1 (K), R.1, R.1
- new net: C.2, J.1 (P1)
- new net: J.12, R.2
- new net: J.13, R.2
- new net: AE.1 (A), C.1
- new net: C.2, R.2, U.16 (SDIO_DATA_CMD)
- new net: D.2 (A2), J.5 (CLK), R.2
- new net: C.2, U.11 (XTAL_OUT), Y.1
- new net: D.2 (A2), J.2 (DAT3/CD), R.2
- new net: C.2, R.2, U.17 (SDIO_DATA_CLK)
- new net: D.2 (A2), J.3 (CMD), R.2
- new net: C.1, L.2, U.23 (VIN_LDO)
- new net: C.1, U.C2 (VDDI)
- new net: R.2, U.K5 (RSTN)
- new net: R.2, U.M6 (CLK)
- new net: C.2, R.2, U.14 (SDIO_DATA_2)
- new net: C.2, R.2, U.19 (SDIO_DATA_1)
- new net: C.2, R.2, U.15 (SDIO_DATA_3)
- new net: C.2, U.2 (WL_BT_ANT)
- new net: L.1, U.21 (VIN_LDO_OUT)
- new net: U.30 (NC), U.32 (NC), U.35 (NC), U.37 (NC), U.38 (NC), U.39 (NC), U.40 (NC), U.5 (NC), U.8 (NC)
- new net: D.2 (A2), J.8 (DAT1), R.2
- new net +1V0: U.28 (DVDD10), U.3 (AVDD10), U.36 (DVDD10), U.40 (AVDD10), U.9 (AVDD10)
- new net 32KIN: U.24 (LPO), X.3 (OUT)
- new net BT_HOST_WAKE_L: U.7 (BT_HOST_WAKE)
- new net BT_RST: U.34 (BT_REG_ON)
- new net BT_WAKE_L: U.6 (BT_WAKE)
- new net DDC_SCL: J.15 (SCL), Q.3 (D), R.2
- new net DDC_SDA: J.16 (SDA), Q.3 (D), R.2
- new net EMMC_CLK: R.1
- new net EMMC_CMD: R.1, U.M5 (CMD)
- new net EMMC_D0: R.1, U.A3 (DAT0)
- new net EMMC_D1: R.1, U.A4 (DAT1)
- new net EMMC_D2: R.1, U.A5 (DAT2)
- new net EMMC_D3: R.1, U.B2 (DAT3)
- new net EMMC_D4: R.1, U.B3 (DAT4)
- new net EMMC_D5: R.1, U.B4 (DAT5)
- new net EMMC_D6: R.1, U.B5 (DAT6)
- new net EMMC_D7: R.1, U.B6 (DAT7)
- new net EMMC_STRB: R.2, U.H5 (DATA_STROBE)
- new net HDMI_CEC: Q.2 (S), R.2
- new net HDMI_HPD: D.1 (K), J.19 (HPD), R.1
- new net HDMI_TX0+: J.7 (D0+)
- new net HDMI_TX0-: J.9 (D0-)
- new net HDMI_TX1+: J.4 (D1+)
- new net HDMI_TX1-: J.6 (D1-)
- new net HDMI_TX2+: J.1 (D2+)
- new net HDMI_TX2-: J.3 (D2-)
- new net HDMI_TXC+: J.10 (CK+)
- new net HDMI_TXC-: J.12 (CK-)
- new net I2C3_SCL_HDMI: Q.2 (S), R.2
- new net I2C3_SDA_HDMI: Q.2 (S), R.2
- new net LAN_VCC: J.14, L.2, R.1, R.1, R.1, R.1, U.38 (ENSWREG), U.44 (VDDREG), U.45 (VDDREG)
- new net LED0_AD0: R.1, U.34 (LED0/PHY_AD0)
- new net LED1_AD1: J.11, U.35 (LED1/PHY_AD1)
- new net LED2_RXDLY: R.1, U.32 (LED2/RXDLY)
- new net MAC_CLK: R.2
- new net MAC_MDC: U.30 (MDC)
- new net MAC_MDIO: U.31 (MDIO)
- new net MAC_RXCLK: R.2
- new net MAC_RXD0: R.2
- new net MAC_RXD1: R.2
- new net MAC_RXD2: R.2
- new net MAC_RXD3: R.2
- new net MAC_RXDV: R.2
- new net PCEC: J.13 (CEC), Q.3 (D), R.2
- new net PHY_CLKOUT125: R.1, U.46 (CLK125)
- new net PHY_INT: R.2, U.20 (INT)
- new net PHY_PMEB: R.2, U.33 (PME)
- new net PHY_RXCLK: R.1, U.19 (RXC)
- new net PHY_RXD0: R.1, U.14 (RXD0)
- new net PHY_RXD1: R.1, R.1, U.16 (RXD1/TXDLY)
- new net PHY_RXD2: R.1, R.2, U.17 (RXD2/AN0)
- new net PHY_RXD3: R.1, R.2, U.18 (RXD3/AN1)
- new net PHY_RXDV: R.1, R.1, U.13 (RXCTL)
- new net PHY_TXCLK: R.2, U.22 (TXC)
- new net PHY_TXD0: R.2, U.23 (TXD0)
- new net PHY_TXD1: R.2, U.24 (TXD1)
- new net PHY_TXD2: R.2, U.25 (TXD2)
- new net PHY_TXD3: R.2, U.26 (TXD3)
- new net PHY_TXEN: U.27 (TXCTL)
- new net RSET: U.39 (RSET)
- new net SDIO_CLK: R.1
- new net SDIO_D0: R.1
- new net SDIO_D1: R.1
- new net SDMMC_CLK: R.1
- new net SDMMC_CMD: R.1
- new net SDMMC_D0: R.1
- new net SDMMC_D1: R.1
- new net SDMMC_D2: R.1
- new net SDMMC_D3: R.1
- new net SDMMC_DET: D.2 (A2), J.9 (DET_B)
- new net TD0+: D.2 (A2), J.2 (P2), U.1 (MDIP0)
- new net TD0-: D.2 (A2), J.3 (P3), U.2 (MDIN0)
- new net TD1+: D.2 (A2), J.4 (P4), U.4 (MDIP1)
- new net TD1-: D.2 (A2), J.7 (P7), U.5 (MDIN1)
- new net TD2+: D.2 (A2), J.5 (P5), U.7 (MDIP2)
- new net TD2-: D.2 (A2), J.6 (P6), U.8 (MDIN2)
- new net TD3+: D.2 (A2), J.8 (P8), U.10 (MDIP3)
- new net TD3-: D.2 (A2), J.9 (P9), U.11 (MDIN3)
- new net UART0_CTS: U.41 (UART_RTS_N)
- new net UART0_RTS: U.44 (UART_CTS_N)
- new net UART0_RX: U.42 (UART_TXD)
- new net UART0_TX: U.43 (UART_RXD)
- new net WORK_LED: R.1
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Other:
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